File: main_board/_autosave-main_board.sch (KiCad schematic (older format))
At the start: 132 parts, among them J1 stepper 0, J10 24VDC output 5, J11 5VDC output 0, J12 5VDC output 1, J13 5VDC output 2, J14 5VDC output 3, J15 5VDC output 4, J16 5VDC output 5, J17 temperature measure 0, J18 temperature measure 1, J19 I2C, J2 stepper 1, J20 I2C, J21 I2C, J22 I2C, J23 hall measure 0, J24 weight measure 0, J25 light measure 0, J26 24VDC_in, J27 24VDC to 5VDC step down, J28 24VDC, J29 24VDC, J3 stepper 2, J30 24VDC, J31 5VDC, J32 5VDC, J33 5VDC, J34 hall measure 1, J35 reflective sensor 0, J36 24VDC, J37 24VDC, J38 24VDC, J39 5VDC, J4 stepper 3, J40 5VDC, J41 5VDC, J42 Conn_01x05_Male, J5 24VDC output 0, J6 24VDC output 1, J7 24VDC output 2, J8 24VDC output 3, J9 24VDC output 4, Q1 Q_NMOS_GDS, Q10 BS170, Q11 BS170, Q12 BS170, Q2 Q_NMOS_GDS, Q3 Q_NMOS_GDS, Q4 Q_NMOS_GDS, Q5 Q_NMOS_GDS, Q6 Q_NMOS_GDS, Q7 BS170, Q8 BS170, Q9 BS170, U1 ESP32-DEVKITC-32D, U2 PCA9685PW

Commit message: making pcb smaller
Parts:
- D13, D14: footprint Diode_SMD:D_SMA_Handsoldering -> Diode_THT:D_A-405_P2.54mm_Vertical_AnodeUp
- J10, J11, J12, J13, J14, J15, J16, J17, J18, J26, J5, J6, J7, J8, J9: footprint TerminalBlock_4Ucon:TerminalBlock_4Ucon_1x02_P3.50mm_Horizontal -> TerminalBlock:TerminalBlock_bornier-2_P5.08mm
Changed lines of the file:
@@
 F 0 "J26" V 13064 512 50  0000 R CNN
 F 1 "24VDC_in" V 12973 512 50  0000 R CNN
-F 2 "TerminalBlock_4Ucon:TerminalBlock_4Ucon_1x02_P3.50mm_Horizontal" H 13100 700 50  0001 C CNN
+F 2 "TerminalBlock:TerminalBlock_bornier-2_P5.08mm" H 13100 700 50  0001 C CNN
 F 3 "~" H 13100 700 50  0001 C CNN
 	1    13100 700
@@
 F 0 "J10" H 4430 8492 50  0000 L CNN
 F 1 "24VDC output 5" H 4430 8401 50  0000 L CNN
-F 2 "TerminalBlock_4Ucon:TerminalBlock_4Ucon_1x02_P3.50mm_Horizontal" H 4350 8500 50  0001 C CNN
+F 2 "TerminalBlock:TerminalBlock_bornier-2_P5.08mm" H 4350 8500 50  0001 C CNN
 F 3 "~" H 4350 8500 50  0001 C CNN
 	1    4350 8500
@@
 F 0 "J9" H 4430 6992 50  0000 L CNN
 F 1 "24VDC output 4" H 4430 6901 50  0000 L CNN
-F 2 "TerminalBlock_4Ucon:TerminalBlock_4Ucon_1x02_P3.50mm_Horizontal" H 4350 7000 50  0001 C CNN
+F 2 "TerminalBlock:TerminalBlock_bornier-2_P5.08mm" H 4350 7000 50  0001 C CNN
 F 3 "~" H 4350 7000 50  0001 C CNN
 	1    4350 7000
@@
 F 0 "J8" H 4430 5492 50  0000 L CNN
 F 1 "24VDC output 3" H 4430 5401 50  0000 L CNN
-F 2 "TerminalBlock_4Ucon:TerminalBlock_4Ucon_1x02_P3.50mm_Horizontal" H 4350 5500 50  0001 C CNN
+F 2 "TerminalBlock:TerminalBlock_bornier-2_P5.08mm" H 4350 5500 50  0001 C CNN
 F 3 "~" H 4350 5500 50  0001 C CNN
 	1    4350 5500
@@
 F 0 "J7" H 4430 3992 50  0000 L CNN
 F 1 "24VDC output 2" H 4430 3901 50  0000 L CNN
-F 2 "TerminalBlock_4Ucon:TerminalBlock_4Ucon_1x02_P3.50mm_Horizontal" H 4350 4000 50  0001 C CNN
+F 2 "TerminalBlock:TerminalBlock_bornier-2_P5.08mm" H 4350 4000 50  0001 C CNN
 F 3 "~" H 4350 4000 50  0001 C CNN
 	1    4350 4000
@@
 F 0 "J6" H 4430 2492 50  0000 L CNN
 F 1 "24VDC output 1" H 4430 2401 50  0000 L CNN
-F 2 "TerminalBlock_4Ucon:TerminalBlock_4Ucon_1x02_P3.50mm_Horizontal" H 4350 2500 50  0001 C CNN
+F 2 "TerminalBlock:TerminalBlock_bornier-2_P5.08mm" H 4350 2500 50  0001 C CNN
 F 3 "~" H 4350 2500 50  0001 C CNN
 	1    4350 2500
@@
 F 0 "J5" H 4430 992 50  0000 L CNN
 F 1 "24VDC output 0" H 4430 901 50  0000 L CNN
-F 2 "TerminalBlock_4Ucon:TerminalBlock_4Ucon_1x02_P3.50mm_Horizontal" H 4350 1000 50  0001 C CNN
+F 2 "TerminalBlock:TerminalBlock_bornier-2_P5.08mm" H 4350 1000 50  0001 C CNN
 F 3 "~" H 4350 1000 50  0001 C CNN
 	1    4350 1000
@@
 F 0 "D13" V 13104 1380 50  0000 L CNN
 F 1 "1N4007" V 13195 1380 50  0000 L CNN
-F 2 "Diode_SMD:D_SMA_Handsoldering" H 13150 1125 50  0001 C CNN
+F 2 "Diode_THT:D_A-405_P2.54mm_Vertical_AnodeUp" H 13150 1125 50  0001 C CNN
 F 3 "http://www.vishay.com/docs/88503/1n4001.pdf" H 13150 1300 50  0001 C CNN
 	1    13150 1300
@@
 F 0 "D14" V 14804 930 50  0000 L CNN
 F 1 "1N4007" V 14895 930 50  0000 L CNN
-F 2 "Diode_SMD:D_SMA_Handsoldering" H 14850 675 50  0001 C CNN
+F 2 "Diode_THT:D_A-405_P2.54mm_Vertical_AnodeUp" H 14850 675 50  0001 C CNN
 F 3 "http://www.vishay.com/docs/88503/1n4001.pdf" H 14850 850 50  0001 C CNN
 	1    14850 850
@@
 F 0 "J17" H 10730 4742 50  0000 L CNN
 F 1 "temperature measure 0" H 10730 4651 50  0000 L CNN
-F 2 "TerminalBlock_4Ucon:TerminalBlock_4Ucon_1x02_P3.50mm_Horizontal" H 10650 4750 50  0001 C CNN
+F 2 "TerminalBlock:TerminalBlock_bornier-2_P5.08mm" H 10650 4750 50  0001 C CNN
 F 3 "~" H 10650 4750 50  0001 C CNN
 	1    10650 4750
@@
 F 0 "J18" H 10730 5492 50  0000 L CNN
 F 1 "temperature measure 1" H 10730 5401 50  0000 L CNN
-F 2 "TerminalBlock_4Ucon:TerminalBlock_4Ucon_1x02_P3.50mm_Horizontal" H 10650 5500 50  0001 C CNN
+F 2 "TerminalBlock:TerminalBlock_bornier-2_P5.08mm" H 10650 5500 50  0001 C CNN
 F 3 "~" H 10650 5500 50  0001 C CNN
 	1    10650 5500
@@
 F 0 "J11" H 6380 992 50  0000 L CNN
 F 1 "5VDC output 0" H 6380 901 50  0000 L CNN
-F 2 "TerminalBlock_4Ucon:TerminalBlock_4Ucon_1x02_P3.50mm_Horizontal" H 6300 1000 50  0001 C CNN
+F 2 "TerminalBlock:TerminalBlock_bornier-2_P5.08mm" H 6300 1000 50  0001 C CNN
 F 3 "~" H 6300 1000 50  0001 C CNN
 	1    6300 1000
@@
 F 0 "J12" H 6380 2492 50  0000 L CNN
 F 1 "5VDC output 1" H 6380 2401 50  0000 L CNN
-F 2 "TerminalBlock_4Ucon:TerminalBlock_4Ucon_1x02_P3.50mm_Horizontal" H 6300 2500 50  0001 C CNN
+F 2 "TerminalBlock:TerminalBlock_bornier-2_P5.08mm" H 6300 2500 50  0001 C CNN
 F 3 "~" H 6300 2500 50  0001 C CNN
 	1    6300 2500
@@
 F 0 "J13" H 6380 3992 50  0000 L CNN
 F 1 "5VDC output 2" H 6380 3901 50  0000 L CNN
-F 2 "TerminalBlock_4Ucon:TerminalBlock_4Ucon_1x02_P3.50mm_Horizontal" H 6300 4000 50  0001 C CNN
+F 2 "TerminalBlock:TerminalBlock_bornier-2_P5.08mm" H 6300 4000 50  0001 C CNN
 F 3 "~" H 6300 4000 50  0001 C CNN
 	1    6300 4000
@@
 F 0 "J14" H 6380 5492 50  0000 L CNN
 F 1 "5VDC output 3" H 6380 5401 50  0000 L CNN
-F 2 "TerminalBlock_4Ucon:TerminalBlock_4Ucon_1x02_P3.50mm_Horizontal" H 6300 5500 50  0001 C CNN
+F 2 "TerminalBlock:TerminalBlock_bornier-2_P5.08mm" H 6300 5500 50  0001 C CNN
 F 3 "~" H 6300 5500 50  0001 C CNN
 	1    6300 5500
@@
 F 0 "J15" H 6380 6992 50  0000 L CNN
 F 1 "5VDC output 4" H 6380 6901 50  0000 L CNN
-F 2 "TerminalBlock_4Ucon:TerminalBlock_4Ucon_1x02_P3.50mm_Horizontal" H 6300 7000 50  0001 C CNN
+F 2 "TerminalBlock:TerminalBlock_bornier-2_P5.08mm" H 6300 7000 50  0001 C CNN
 F 3 "~" H 6300 7000 50  0001 C CNN
 	1    6300 7000
@@
 F 0 "J16" H 6380 8492 50  0000 L CNN
 F 1 "5VDC output 5" H 6380 8401 50  0000 L CNN
-F 2 "TerminalBlock_4Ucon:TerminalBlock_4Ucon_1x02_P3.50mm_Horizontal" H 6300 8500 50  0001 C CNN
+F 2 "TerminalBlock:TerminalBlock_bornier-2_P5.08mm" H 6300 8500 50  0001 C CNN
 F 3 "~" H 6300 8500 50  0001 C CNN
 	1    6300 8500
