File: main_board/main_board.sch (KiCad schematic (older format))
At the start: 33 parts, among them J1 Conn_01x04_Male, J2 Conn_01x04_Male, J3 Conn_01x04_Male, J4 Conn_01x04_Male, J5 Screw_Terminal_01x02, J6 Screw_Terminal_01x04, J7 Screw_Terminal_01x02, J8 Screw_Terminal_01x04, J9 Screw_Terminal_01x02, Q1 Q_NMOS_GDS, Q2 Q_NMOS_GDS, U1 ESP32-DEVKITC-32D, U2 PCF8575PWE4

Commit message: added parts to scheme
Parts:
- removed J6, J8: Screw_Terminal_01x04, TerminalBlock:TerminalBlock_Altech_AK300-4_P5.00mm, symbol Connector:Screw_Terminal_01x04
- removed U2: PCF8575PWE4, PCF8575PWE4:SOP65P640X120-24N, symbol PCF8575PWE4:PCF8575PWE4
- added C10, C5, C6, C7, C8, C9: C, symbol Device:C
- added D3, D4, D5, D6: 1N4007, Diode_THT:D_DO-41_SOD81_P10.16mm_Horizontal, symbol Diode:1N4007
- added F1: Fuse, symbol Device:Fuse
- added J10, J14, J15, J16, J6, J8: Conn_01x02_Female, symbol Connector:Conn_01x02_Female
- added J11, J12, J13, J17, J18: Screw_Terminal_01x02, TerminalBlock:TerminalBlock_Altech_AK300-2_P5.00mm, symbol Connector:Screw_Terminal_01x02
- added J19, J20: Conn_01x03_Male, symbol Connector:Conn_01x03_Male
- added J21: Conn_01x05_Female, symbol Connector:Conn_01x05_Female
- added J22, J24, J25, J26, J27: Conn_01x04_Female, symbol Connector:Conn_01x04_Female
- added J23: power_input, symbol Connector:Screw_Terminal_01x02
- added Q3, Q4, Q5, Q6: Q_NMOS_GDS, Package_TO_SOT_THT:TO-220-3_Vertical, symbol Device:Q_NMOS_GDS
- added R11, R13, R15, R17: 3k3, Resistor_SMD:R_1206_3216Metric_Pad1.30x1.75mm_HandSolder, symbol Device:R
- added R12, R14, R16, R18: 10k, Resistor_SMD:R_1206_3216Metric_Pad1.30x1.75mm_HandSolder, symbol Device:R
- added R19, R20, R21, R22, R23, R24, R25: R, symbol Device:R
- added SW1: Rotary_Encoder_Switch, symbol Device:Rotary_Encoder_Switch
- added U2: PCA9685PW, Package_SO:TSSOP-28_4.4x9.7mm_P0.65mm, symbol Driver_LED:PCA9685PW
- U1: symbol ESP32-DEVKITC-32D:ESP32-DEVKITC-32D -> main_board-rescue:ESP32-DEVKITC-32D-ESP32-DEVKITC-32D
Connections:
- net labels added: +5V, AO, CLK, DT, GND, SCK, SI, button, enca, encb, hallmeasure1, hallmeasure2, output1, output2, output3, output4, output5, output6, reflectivesensor1, reflectivesensor2
- net labels removed: +3.3V, GND1, GND2, filamentDimMeasure1, filamentDimMeasure2, heater1, heater2and3, potMeasure
- wire segments 164 -> 245
- no-connect marks 4 -> 1
Other:
- moved on the sheet: J7, J9, R5, R6, R7, R8

Commit message: schematic update
Parts:
- removed C10: C, symbol Device:C
- removed J7, J9: Screw_Terminal_01x02, TerminalBlock:TerminalBlock_Altech_AK300-2_P5.00mm, symbol Connector:Screw_Terminal_01x02
- removed R25: R, symbol Device:R
- removed R6: 100k, Resistor_SMD:R_1206_3216Metric_Pad1.30x1.75mm_HandSolder, symbol Device:R
- added C11: 100uF, symbol Device:C
- added C12, C13, C14: 100n, symbol Device:C
- added C? (x2): C, symbol Device:C
- added D7, D9: 1N4007, Diode_THT:D_DO-41_SOD81_P10.16mm_Horizontal, symbol Diode:1N4007
- added D8: LED, symbol Device:LED
- added J28: 24VDC to 5VDC step down, symbol Connector:Conn_01x04_Male
- added J?: reflective sensor 0, symbol Connector:Conn_01x04_Female
- added J? (x6): 5VDC, symbol Connector:Conn_01x02_Female
- added J?: temperature measure 0, symbol Connector:Conn_01x02_Female
- added J?: temperature measure 1, symbol Connector:Conn_01x02_Female
- added R? (x2): 100R, symbol Device:R
- added R?: 100k, symbol Device:R
- added R? (x2): R, symbol Device:R
- added R?: 390R, symbol Device:R
- added R?: 100k, Resistor_SMD:R_1206_3216Metric_Pad1.30x1.75mm_HandSolder, symbol Device:R
- C1, C2, C3, C4: value CP -> 100uF
- J1: value Conn_01x04_Male -> stepper 0
- J10, J14, J15, J16, J6, J8: value Conn_01x02_Female -> 24VDC
- J11: value Screw_Terminal_01x02 -> 24VDC output 1
- J12: value Screw_Terminal_01x02 -> 24VDC output 2
- J13: value Screw_Terminal_01x02 -> 24VDC output 3
- J17: value Screw_Terminal_01x02 -> 24VDC output 4
- J18: value Screw_Terminal_01x02 -> 24VDC output 5
- J19: value Conn_01x03_Male -> hall measure 1
- J2: value Conn_01x04_Male -> stepper 1
- J20: value Conn_01x03_Male -> hall measure 0
- J21: value Conn_01x05_Female -> light measure 0
- J22: value Conn_01x04_Female -> weight measure 0
- J23: value power_input -> 24VDC_in
- J24: value Conn_01x04_Female -> I2C 0
- J25: value Conn_01x04_Female -> I2C 2
- J26: value Conn_01x04_Female -> I2C 1
- J27: value Conn_01x04_Female -> I2C 3
- J3: value Conn_01x04_Male -> stepper 2
- J4: value Conn_01x04_Male -> stepper 3
- J5: value Screw_Terminal_01x02 -> 24VDC output 0
- R22: value R -> 150R
Connections:
- net DIR4 is gone; now on net DIR3: A4.16 (DIR), U1.10 (IO26)
- net STEP4 is gone; now on net STEP3: A4.15 (STEP), U1.11 (IO27)
- net reflectivesensor2 is gone; now on net OE: U1.9 (IO25)
- net tempMeasure2 is gone; now on net tempMeasure1: R8.2
- net +24V: now also D7.1 (K), J28.3 (Pin_3), R?.1
- net +5V: now also C11.1, D8.2 (A), D9.1 (K), J28.1 (Pin_1), J?.2 (Pin_2), J?.2 (Pin_2), J?.2 (Pin_2), J?.2 (Pin_2), J?.2 (Pin_2), J?.2 (Pin_2); no longer R10.1, R5.1, R9.1, SW1.S2
- net DIR1: now also A2.16 (DIR), U1.13 (IO12); no longer A1.16 (DIR), U1.33 (IO0)
- net DIR2: now also A3.16 (DIR), U1.27 (IO19); no longer A2.16 (DIR), U1.13 (IO12)
- net DIR3: no longer A3.16 (DIR), U1.27 (IO19)
- net GND: now also R22.2, C13.1, C14.2, C?.1, C?.2, D7.2 (A), D9.2 (A), J28.2 (Pin_2), J?.1 (Pin_1), J?.1 (Pin_1), J?.1 (Pin_1), J?.1 (Pin_1), J?.1 (Pin_1), J?.1 (Pin_1), J?.1 (Pin_1), J?.1 (Pin_1), J?.1 (Pin_1), J?.2 (Pin_2), R?.2
- net STEP1: now also A2.15 (STEP), U1.30 (IO17); no longer A1.15 (STEP), U1.29 (IO5)
- net STEP2: now also A3.15 (STEP), U1.21 (IO23); no longer A2.15 (STEP), U1.30 (IO17)
- net STEP3: no longer A3.15 (STEP), U1.21 (IO23)
- net button: now also SW1.S2, C12.2; no longer R22.1
- net enca: now also C14.1
- net encb: now also C13.2
- net hallmeasure1: now also U1.15 (IO13); no longer U1.3 (SENSOR_VP)
- net stepperErr: now also U2.18 (LED11); no longer U2.13 (LED7)
- net stepperON: now also U2.17 (LED10); no longer U2.12 (LED6)
- net tempMeasure1: now also C?.1, R?.2; no longer C9.1, R24.2, R7.2
- net at R24.1, R5.2: now also J?.2 (Pin_2)
- net at U1.19 (EXT_5V): now also C11.2
- net +3V3: now reaches SW1.S1
- net +3V3: now also R10.1, R5.1, R9.1, C12.1, R?.1, R?.1; no longer R22.2
- net 5VDC_output2: now reaches U2.15 (LED8)
- net 5VDC_output3: now reaches U2.16 (LED9)
- net LEDcon0: now reaches U2.19 (LED12)
- net LEDcon0: now also R?.1
- net OE: now reaches U2.23 (~OE)
- net hallmeasure2 renamed hallmeasure0
- net hallmeasure0: now also U1.3 (SENSOR_VP); no longer U1.15 (IO13)
- net output1 renamed 24VDC_output0
- net output2 renamed 24VDC_output1
- net output3 renamed 24VDC_output2
- net output4 renamed 24VDC_output3
- net output5 renamed 24VDC_output4
- net output6 renamed 24VDC_output5
- net reflectivesensor1 renamed reflectivesensor0
- net reflectivesensor0: now also C?.2, R?.2
- new net: J28.4 (Pin_4), R?.1, R?.2
- new net: D8.1 (K), R22.1
- new net: J?.3 (Pin_3), R?.1, R?.2
- new net: J?.4 (Pin_4), R?.2
- new net: J?.2 (Pin_2), R?.1, R?.2
- new net 5VDC_output0: U2.12 (LED6)
- new net 5VDC_output1: U2.13 (LED7)
- new net DIR0: A1.16 (DIR), U1.33 (IO0)
- new net STEP0: A1.15 (STEP), U1.29 (IO5)
- new net tempMeasure0: C9.1, R24.2, R7.2
Other:
- moved on the sheet: A1, C1, C5, C6, C7, C8, C9, D5, D6, F1, J1, J10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

Commit message: footprints assigned
Parts:
- removed J?: temperature measure 0, symbol Connector:Conn_01x02_Female
- removed J?: temperature measure 1, symbol Connector:Conn_01x02_Female
- removed R?: 390R, symbol Device:R
- removed R?: 100R, symbol Device:R
- removed R?: R, symbol Device:R
- added C5: 10uF, Capacitor_THT:CP_Radial_D4.0mm_P1.50mm, symbol Device:C
- added D10, D11, D12, D7, D8, D9: 1N4007, Diode_THT:D_DO-41_SOD81_P10.16mm_Horizontal, symbol Diode:1N4007
- added J11: 5VDC output 0, TerminalBlock_4Ucon:TerminalBlock_4Ucon_1x02_P3.50mm_Horizontal, symbol Connector:Screw_Terminal_01x02
- added J12: 5VDC output 1, TerminalBlock_4Ucon:TerminalBlock_4Ucon_1x02_P3.50mm_Horizontal, symbol Connector:Screw_Terminal_01x02
- added J13: 5VDC output 2, TerminalBlock_4Ucon:TerminalBlock_4Ucon_1x02_P3.50mm_Horizontal, symbol Connector:Screw_Terminal_01x02
- added J14: 5VDC output 3, TerminalBlock_4Ucon:TerminalBlock_4Ucon_1x02_P3.50mm_Horizontal, symbol Connector:Screw_Terminal_01x02
- added J15: 5VDC output 4, TerminalBlock_4Ucon:TerminalBlock_4Ucon_1x02_P3.50mm_Horizontal, symbol Connector:Screw_Terminal_01x02
- added J16: 5VDC output 5, TerminalBlock_4Ucon:TerminalBlock_4Ucon_1x02_P3.50mm_Horizontal, symbol Connector:Screw_Terminal_01x02
- added J17: temperature measure 0, TerminalBlock:TerminalBlock_Altech_AK300-2_P5.00mm, symbol Connector:Screw_Terminal_01x02
- added J18: temperature measure 1, TerminalBlock:TerminalBlock_Altech_AK300-2_P5.00mm, symbol Connector:Screw_Terminal_01x02
- added Q10, Q11, Q12, Q7, Q8, Q9: BS170, Package_TO_SOT_THT:TO-92_Inline_Wide, symbol Transistor_FET:BS170
- added R13, R15, R17, R21: 3k3, Resistor_SMD:R_1206_3216Metric_Pad1.30x1.75mm_HandSolder, symbol Device:R
- added R14, R16, R18, R22, R31, R32, R33, R35, R37: 10k, Resistor_SMD:R_1206_3216Metric_Pad1.30x1.75mm_HandSolder, symbol Device:R
- C1, C2, C3, C4: footprint Capacitor_THT:CP_Radial_D8.0mm_P3.50mm -> Capacitor_THT:CP_Radial_D6.3mm_P2.50mm
- C10: renamed from C7; value C -> 100uF; footprint (none) -> Capacitor_THT:CP_Radial_D6.3mm_P2.50mm
- C11: renamed from C8; value C -> 100uF; footprint (none) -> Capacitor_THT:CP_Radial_D6.3mm_P2.50mm
- C12: renamed from C13; footprint (none) -> Capacitor_SMD:C_0603_1608Metric_Pad1.08x0.95mm_HandSolder
- C13: renamed from C14; footprint (none) -> Capacitor_SMD:C_0603_1608Metric_Pad1.08x0.95mm_HandSolder
- C14: renamed from C11; footprint (none) -> Capacitor_THT:CP_Radial_D6.3mm_P2.50mm
- C15: renamed from C5; value C -> 100uF; footprint (none) -> Capacitor_THT:CP_Radial_D6.3mm_P2.50mm
- C16, C7: renamed from C?; value C -> 100uF; footprint (none) -> Capacitor_THT:CP_Radial_D6.3mm_P2.50mm
- C6: renamed from C9; value C -> 100uF; footprint (none) -> Capacitor_THT:CP_Radial_D6.3mm_P2.50mm
- C8: renamed from C12; footprint (none) -> Capacitor_SMD:C_0603_1608Metric_Pad1.08x0.95mm_HandSolder
- C9: renamed from C6; value C -> 100uF; footprint (none) -> Capacitor_THT:CP_Radial_D6.3mm_P2.50mm
- D15: renamed from D8; footprint (none) -> LED_THT:LED_D3.0mm
- F1: footprint (none) -> Fuse:Fuseholder_Cylinder-5x20mm_Schurter_0031_8201_Horizontal_Open
- J10: renamed from J18; footprint TerminalBlock:TerminalBlock_Altech_AK300-2_P5.00mm -> TerminalBlock_4Ucon:TerminalBlock_4Ucon_1x02_P3.50mm_Horizontal
- J19: renamed from J24; footprint (none) -> Connector_PinHeader_2.54mm:PinHeader_1x04_P2.54mm_Vertical
- J20: renamed from J25; footprint (none) -> Connector_PinHeader_2.54mm:PinHeader_1x04_P2.54mm_Vertical
- J21: renamed from J26; footprint (none) -> Connector_PinHeader_2.54mm:PinHeader_1x04_P2.54mm_Vertical
- J22: renamed from J27; footprint (none) -> Connector_PinHeader_2.54mm:PinHeader_1x04_P2.54mm_Vertical
- J23: renamed from J20; footprint (none) -> Connector_PinHeader_2.54mm:PinHeader_1x03_P2.54mm_Vertical
- J24: renamed from J22; footprint (none) -> Connector_PinHeader_2.54mm:PinHeader_1x04_P2.54mm_Vertical
- J25: renamed from J21; footprint (none) -> Connector_PinHeader_2.54mm:PinHeader_1x05_P2.54mm_Vertical
- J26: renamed from J23; footprint (none) -> TerminalBlock_4Ucon:TerminalBlock_4Ucon_1x02_P3.50mm_Horizontal
- J27: renamed from J28; footprint (none) -> Connector_PinHeader_2.54mm:PinHeader_1x04_P2.54mm_Vertical
- J28: renamed from J6; footprint (none) -> Connector_PinHeader_2.54mm:PinHeader_1x02_P2.54mm_Vertical
- J29: renamed from J8; footprint (none) -> Connector_PinHeader_2.54mm:PinHeader_1x02_P2.54mm_Vertical
- J30: renamed from J10; footprint (none) -> Connector_PinHeader_2.54mm:PinHeader_1x02_P2.54mm_Vertical
- J31, J32, J33, J39, J40, J41: renamed from J?; footprint (none) -> Connector_PinHeader_2.54mm:PinHeader_1x02_P2.54mm_Vertical
- J34: renamed from J19; footprint (none) -> Connector_PinHeader_2.54mm:PinHeader_1x03_P2.54mm_Vertical
- J35: renamed from J?; footprint (none) -> Connector_PinHeader_2.54mm:PinHeader_1x04_P2.54mm_Vertical
- J36: renamed from J14; footprint (none) -> Connector_PinHeader_2.54mm:PinHeader_1x02_P2.54mm_Vertical
- J37: renamed from J15; footprint (none) -> Connector_PinHeader_2.54mm:PinHeader_1x02_P2.54mm_Vertical
- J38: renamed from J16; footprint (none) -> Connector_PinHeader_2.54mm:PinHeader_1x02_P2.54mm_Vertical
- J5: footprint TerminalBlock:TerminalBlock_Altech_AK300-2_P5.00mm -> TerminalBlock_4Ucon:TerminalBlock_4Ucon_1x02_P3.50mm_Horizontal
- J6: renamed from J11; footprint TerminalBlock:TerminalBlock_Altech_AK300-2_P5.00mm -> TerminalBlock_4Ucon:TerminalBlock_4Ucon_1x02_P3.50mm_Horizontal
- J7: renamed from J12; footprint TerminalBlock:TerminalBlock_Altech_AK300-2_P5.00mm -> TerminalBlock_4Ucon:TerminalBlock_4Ucon_1x02_P3.50mm_Horizontal
- J8: renamed from J13; footprint TerminalBlock:TerminalBlock_Altech_AK300-2_P5.00mm -> TerminalBlock_4Ucon:TerminalBlock_4Ucon_1x02_P3.50mm_Horizontal
- J9: renamed from J17; footprint TerminalBlock:TerminalBlock_Altech_AK300-2_P5.00mm -> TerminalBlock_4Ucon:TerminalBlock_4Ucon_1x02_P3.50mm_Horizontal
- R19, R23: value R -> 3k3; footprint (none) -> Resistor_SMD:R_1206_3216Metric_Pad1.30x1.75mm_HandSolder
- R20, R24: value R -> 10k; footprint (none) -> Resistor_SMD:R_1206_3216Metric_Pad1.30x1.75mm_HandSolder
- R34: renamed from R21; value R -> 10k; footprint (none) -> Resistor_SMD:R_1206_3216Metric_Pad1.30x1.75mm_HandSolder
- R36, R40: renamed from R?; footprint (none) -> Resistor_SMD:R_1206_3216Metric_Pad1.30x1.75mm_HandSolder
- R38: renamed from R?; value R -> 10k; footprint (none) -> Resistor_SMD:R_1206_3216Metric_Pad1.30x1.75mm_HandSolder
- R39: renamed from R22; footprint (none) -> Resistor_SMD:R_1206_3216Metric_Pad1.30x1.75mm_HandSolder
- SW1: footprint (none) -> Rotary_Encoder:RotaryEncoder_Alps_EC11E-Switch_Vertical_H20mm
- gave numbers to parts that had none: 1
- renumbered D7 to D13, D9 to D14, R16 to R10, R17 to R11, R18 to R12, R7 to R25, R8 to R26, R5 to R27, R9 to R29, R10 to R30, R11 to R5, R12 to R6, R13 to R7, R14 to R8, R15 to R9
Connections:
- net +5V: now also C14.2, U1.19 (EXT_5V), C5.1, D10.1 (K), D11.1 (K), D12.1 (K), D7.1 (K), D8.1 (K), D9.1 (K), J11.1 (Pin_1), J12.1 (Pin_1), J13.1 (Pin_1), J14.1 (Pin_1), J15.1 (Pin_1), J16.1 (Pin_1); no longer C14.1
- net 5VDC_output0: now also R19.2, R20.2, R23.2, R24.2, R13.2, R14.2, R15.2, R16.2, R17.2, R18.2, R21.2, R22.2
- net AO: now also R34.1; no longer R34.2
- net DT: now also R35.1; no longer R23.2
- net GND: now also C14.1, R20.1, R24.1, C5.2, J17.1 (Pin_1), J18.1 (Pin_1), Q10.3 (S), Q11.3 (S), Q12.3 (S), Q7.3 (S), Q8.3 (S), Q9.3 (S), R14.1, R16.1, R18.1, R22.1
- net hallmeasure0: now also R33.2; no longer R20.2
- net hallmeasure1: now also R37.2; no longer R19.2
- net tempMeasure0: now also R31.1; no longer R24.2
- net tempMeasure1: now also R32.1
- net at R27.2: now also J17.2 (Pin_2), R31.2; no longer R24.1
- net at J34.3 (Pin_3): now also R37.1; no longer R19.1
- net at J23.3 (Pin_3): now also R33.1; no longer R20.1
- net at J25.2 (Pin_2): now also R34.2; no longer R34.1
- net at J24.3 (Pin_3): now also R35.2; no longer R23.1
- net at R28.2: now also J18.2 (Pin_2), R32.2
- new net: D7.2 (A), J11.2 (Pin_2), Q7.1 (D)
- new net: Q7.2 (G), R13.1
- new net: D8.2 (A), J12.2 (Pin_2), Q8.1 (D)
- new net: Q8.2 (G), R15.1
- new net: D9.2 (A), J13.2 (Pin_2), Q9.1 (D)
- new net: Q9.2 (G), R17.1
- new net: D10.2 (A), J14.2 (Pin_2), Q10.1 (D)
- new net: Q10.2 (G), R19.1
- new net: D11.2 (A), J15.2 (Pin_2), Q11.1 (D)
- new net: Q11.2 (G), R21.1
- new net: D12.2 (A), J16.2 (Pin_2), Q12.1 (D)
- new net: Q12.2 (G), R23.1
Other:
- moved on the sheet: C10, C11, C14, C15, C16, C6, C7, C9, D1, D14, D15, D2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

Commit message: PCB started
Parts:
- D1, D10, D11, D12, D13, D14, D2, D3, D4, D5, D6, D7, D8, D9: footprint Diode_THT:D_DO-41_SOD81_P10.16mm_Horizontal -> Diode_SMD:D_SMA_Handsoldering
- J17, J18: footprint TerminalBlock:TerminalBlock_Altech_AK300-2_P5.00mm -> TerminalBlock_4Ucon:TerminalBlock_4Ucon_1x02_P3.50mm_Horizontal
- J19: value I2C 0 -> I2C
- J20: value I2C 2 -> I2C
- J21: value I2C 1 -> I2C
- J22: value I2C 3 -> I2C
Connections:
- net +3V3: now also U1.1 (3V3)
- net +5V: now also C14.1; no longer C14.2
- net GND: now also C14.2; no longer C14.1
Other:
- moved on the sheet: C14
Changed lines of the file:
@@
 P 11000 1750
 F 0 "J19" H 10892 1325 50  0000 C CNN
-F 1 "I2C 0" H 10892 1416 50  0000 C CNN
+F 1 "I2C" H 10892 1416 50  0000 C CNN
 F 2 "Connector_PinHeader_2.54mm:PinHeader_1x04_P2.54mm_Vertical" H 11000 1750 50  0001 C CNN
 F 3 "~" H 11000 1750 50  0001 C CNN
@@
 P 11000 2400
 F 0 "J20" H 10892 1975 50  0000 C CNN
-F 1 "I2C 2" H 10892 2066 50  0000 C CNN
+F 1 "I2C" H 10892 2066 50  0000 C CNN
 F 2 "Connector_PinHeader_2.54mm:PinHeader_1x04_P2.54mm_Vertical" H 11000 2400 50  0001 C CNN
 F 3 "~" H 11000 2400 50  0001 C CNN
@@
 P 11850 2400
 F 0 "J22" H 11742 1975 50  0000 C CNN
-F 1 "I2C 3" H 11742 2066 50  0000 C CNN
+F 1 "I2C" H 11742 2066 50  0000 C CNN
 F 2 "Connector_PinHeader_2.54mm:PinHeader_1x04_P2.54mm_Vertical" H 11850 2400 50  0001 C CNN
 F 3 "~" H 11850 2400 50  0001 C CNN
@@
 P 11850 1750
 F 0 "J21" H 11742 1325 50  0000 C CNN
-F 1 "I2C 1" H 11742 1416 50  0000 C CNN
+F 1 "I2C" H 11742 1416 50  0000 C CNN
 F 2 "Connector_PinHeader_2.54mm:PinHeader_1x04_P2.54mm_Vertical" H 11850 1750 50  0001 C CNN
 F 3 "~" H 11850 1750 50  0001 C CNN
@@
 L Device:C C14
 U 1 1 629531CD
-P 14600 850
-F 0 "C14" V 14852 850 50  0000 C CNN
-F 1 "100uF" V 14761 850 50  0000 C CNN
-F 2 "Capacitor_THT:CP_Radial_D6.3mm_P2.50mm" H 14638 700 50  0001 C CNN
-F 3 "~" H 14600 850 50  0001 C CNN
-	1    14600 850
-	-1   0    0    1
+P 14450 850
+F 0 "C14" V 14702 850 50  0000 C CNN
+F 1 "100uF" V 14611 850 50  0000 C CNN
+F 2 "Capacitor_THT:CP_Radial_D6.3mm_P2.50mm" H 14488 700 50  0001 C CNN
+F 3 "~" H 14450 850 50  0001 C CNN
+	1    14450 850
+	1    0    0    -1
 $EndComp
 $Comp
@@
 F 0 "D6" V 3804 8630 50  0000 L CNN
 F 1 "1N4007" V 3895 8630 50  0000 L CNN
-F 2 "Diode_THT:D_DO-41_SOD81_P10.16mm_Horizontal" H 3850 8375 50  0001 C CNN
+F 2 "Diode_SMD:D_SMA_Handsoldering" H 3850 8375 50  0001 C CNN
 F 3 "http://www.vishay.com/docs/88503/1n4001.pdf" H 3850 8550 50  0001 C CNN
 	1    3850 8550
@@
 F 0 "D5" V 3804 7130 50  0000 L CNN
 F 1 "1N4007" V 3895 7130 50  0000 L CNN
-F 2 "Diode_THT:D_DO-41_SOD81_P10.16mm_Horizontal" H 3850 6875 50  0001 C CNN
+F 2 "Diode_SMD:D_SMA_Handsoldering" H 3850 6875 50  0001 C CNN
 F 3 "http://www.vishay.com/docs/88503/1n4001.pdf" H 3850 7050 50  0001 C CNN
 	1    3850 7050
@@
 F 0 "D4" V 3804 5630 50  0000 L CNN
 F 1 "1N4007" V 3895 5630 50  0000 L CNN
-F 2 "Diode_THT:D_DO-41_SOD81_P10.16mm_Horizontal" H 3850 5375 50  0001 C CNN
+F 2 "Diode_SMD:D_SMA_Handsoldering" H 3850 5375 50  0001 C CNN
 F 3 "http://www.vishay.com/docs/88503/1n4001.pdf" H 3850 5550 50  0001 C CNN
 	1    3850 5550
@@
 F 0 "D3" V 3804 4130 50  0000 L CNN
 F 1 "1N4007" V 3895 4130 50  0000 L CNN
-F 2 "Diode_THT:D_DO-41_SOD81_P10.16mm_Horizontal" H 3850 3875 50  0001 C CNN
+F 2 "Diode_SMD:D_SMA_Handsoldering" H 3850 3875 50  0001 C CNN
 F 3 "http://www.vishay.com/docs/88503/1n4001.pdf" H 3850 4050 50  0001 C CNN
 	1    3850 4050
@@
 F 0 "D2" V 3804 2630 50  0000 L CNN
 F 1 "1N4007" V 3895 2630 50  0000 L CNN
-F 2 "Diode_THT:D_DO-41_SOD81_P10.16mm_Horizontal" H 3850 2375 50  0001 C CNN
+F 2 "Diode_SMD:D_SMA_Handsoldering" H 3850 2375 50  0001 C CNN
 F 3 "http://www.vishay.com/docs/88503/1n4001.pdf" H 3850 2550 50  0001 C CNN
 	1    3850 2550
@@
 F 0 "D1" V 3804 1130 50  0000 L CNN
 F 1 "1N4007" V 3895 1130 50  0000 L CNN
-F 2 "Diode_THT:D_DO-41_SOD81_P10.16mm_Horizontal" H 3850 875 50  0001 C CNN
+F 2 "Diode_SMD:D_SMA_Handsoldering" H 3850 875 50  0001 C CNN
 F 3 "http://www.vishay.com/docs/88503/1n4001.pdf" H 3850 1050 50  0001 C CNN
 	1    3850 1050
@@
 F 0 "D13" V 13104 1380 50  0000 L CNN
 F 1 "1N4007" V 13195 1380 50  0000 L CNN
-F 2 "Diode_THT:D_DO-41_SOD81_P10.16mm_Horizontal" H 13150 1125 50  0001 C CNN
+F 2 "Diode_SMD:D_SMA_Handsoldering" H 13150 1125 50  0001 C CNN
 F 3 "http://www.vishay.com/docs/88503/1n4001.pdf" H 13150 1300 50  0001 C CNN
 	1    13150 1300
@@
 F 0 "D14" V 14804 930 50  0000 L CNN
 F 1 "1N4007" V 14895 930 50  0000 L CNN
-F 2 "Diode_THT:D_DO-41_SOD81_P10.16mm_Horizontal" H 14850 675 50  0001 C CNN
+F 2 "Diode_SMD:D_SMA_Handsoldering" H 14850 675 50  0001 C CNN
 F 3 "http://www.vishay.com/docs/88503/1n4001.pdf" H 14850 850 50  0001 C CNN
 	1    14850 850
@@
 F 0 "J17" H 10730 4742 50  0000 L CNN
 F 1 "temperature measure 0" H 10730 4651 50  0000 L CNN
-F 2 "TerminalBlock:TerminalBlock_Altech_AK300-2_P5.00mm" H 10650 4750 50  0001 C CNN
+F 2 "TerminalBlock_4Ucon:TerminalBlock_4Ucon_1x02_P3.50mm_Horizontal" H 10650 4750 50  0001 C CNN
 F 3 "~" H 10650 4750 50  0001 C CNN
 	1    10650 4750
@@
 F 0 "J18" H 10730 5492 50  0000 L CNN
 F 1 "temperature measure 1" H 10730 5401 50  0000 L CNN
-F 2 "TerminalBlock:TerminalBlock_Altech_AK300-2_P5.00mm" H 10650 5500 50  0001 C CNN
+F 2 "TerminalBlock_4Ucon:TerminalBlock_4Ucon_1x02_P3.50mm_Horizontal" H 10650 5500 50  0001 C CNN
 F 3 "~" H 10650 5500 50  0001 C CNN
 	1    10650 5500
@@
 	7600 2650 7650 2650
 Wire Wire Line
-	14600 700  14750 700
+	14450 700  14750 700
 Wire Wire Line
-	14600 1000 14750 1000
+	14450 1000 14750 1000
 $Comp
 L power:+5V #PWR086
@@
 F 0 "D7" V 5754 1130 50  0000 L CNN
 F 1 "1N4007" V 5845 1130 50  0000 L CNN
-F 2 "Diode_THT:D_DO-41_SOD81_P10.16mm_Horizontal" H 5800 875 50  0001 C CNN
+F 2 "Diode_SMD:D_SMA_Handsoldering" H 5800 875 50  0001 C CNN
 F 3 "http://www.vishay.com/docs/88503/1n4001.pdf" H 5800 1050 50  0001 C CNN
 	1    5800 1050
@@
 F 0 "D8" V 5754 2630 50  0000 L CNN
 F 1 "1N4007" V 5845 2630 50  0000 L CNN
-F 2 "Diode_THT:D_DO-41_SOD81_P10.16mm_Horizontal" H 5800 2375 50  0001 C CNN
+F 2 "Diode_SMD:D_SMA_Handsoldering" H 5800 2375 50  0001 C CNN
 F 3 "http://www.vishay.com/docs/88503/1n4001.pdf" H 5800 2550 50  0001 C CNN
 	1    5800 2550
@@
 F 0 "D9" V 5754 4130 50  0000 L CNN
 F 1 "1N4007" V 5845 4130 50  0000 L CNN
-F 2 "Diode_THT:D_DO-41_SOD81_P10.16mm_Horizontal" H 5800 3875 50  0001 C CNN
+F 2 "Diode_SMD:D_SMA_Handsoldering" H 5800 3875 50  0001 C CNN
 F 3 "http://www.vishay.com/docs/88503/1n4001.pdf" H 5800 4050 50  0001 C CNN
 	1    5800 4050
@@
 F 0 "D10" V 5754 5630 50  0000 L CNN
 F 1 "1N4007" V 5845 5630 50  0000 L CNN
-F 2 "Diode_THT:D_DO-41_SOD81_P10.16mm_Horizontal" H 5800 5375 50  0001 C CNN
+F 2 "Diode_SMD:D_SMA_Handsoldering" H 5800 5375 50  0001 C CNN
 F 3 "http://www.vishay.com/docs/88503/1n4001.pdf" H 5800 5550 50  0001 C CNN
 	1    5800 5550
@@
 F 0 "D11" V 5754 7130 50  0000 L CNN
 F 1 "1N4007" V 5845 7130 50  0000 L CNN
-F 2 "Diode_THT:D_DO-41_SOD81_P10.16mm_Horizontal" H 5800 6875 50  0001 C CNN
+F 2 "Diode_SMD:D_SMA_Handsoldering" H 5800 6875 50  0001 C CNN
 F 3 "http://www.vishay.com/docs/88503/1n4001.pdf" H 5800 7050 50  0001 C CNN
 	1    5800 7050
@@
 F 0 "D12" V 5754 8630 50  0000 L CNN
 F 1 "1N4007" V 5845 8630 50  0000 L CNN
-F 2 "Diode_THT:D_DO-41_SOD81_P10.16mm_Horizontal" H 5800 8375 50  0001 C CNN
+F 2 "Diode_SMD:D_SMA_Handsoldering" H 5800 8375 50  0001 C CNN
 F 3 "http://www.vishay.com/docs/88503/1n4001.pdf" H 5800 8550 50  0001 C CNN
 	1    5800 8550
@@
 Wire Wire Line
 	15250 6750 15200 6750
+$Comp
+L power:+3.3V #PWR0109
+U 1 1 6486F7DD
+P 7650 850
+F 0 "#PWR0109" H 7650 700 50  0001 C CNN
+F 1 "+3.3V" V 7665 978 50  0000 L CNN
+F 2 "" H 7650 850 50  0001 C CNN
+F 3 "" H 7650 850 50  0001 C CNN
+	1    7650 850
+	0    -1   -1   0
+$EndComp
 $EndSCHEMATC
