File: main_board/main_board.sch (KiCad schematic (older format))
At the start: 132 parts, among them J1 stepper 0, J10 24VDC output 5, J11 5VDC output 0, J12 5VDC output 1, J13 5VDC output 2, J14 5VDC output 3, J15 5VDC output 4, J16 5VDC output 5, J17 temperature measure 0, J18 temperature measure 1, J19 I2C, J2 stepper 1, J20 I2C, J21 I2C, J22 I2C, J23 hall measure 0, J24 weight measure 0, J25 light measure 0, J26 24VDC_in, J27 24VDC to 5VDC step down, J28 24VDC, J29 24VDC, J3 stepper 2, J30 24VDC, J31 5VDC, J32 5VDC, J33 5VDC, J34 hall measure 1, J35 reflective sensor 0, J36 24VDC, J37 24VDC, J38 24VDC, J39 5VDC, J4 stepper 3, J40 5VDC, J41 5VDC, J5 24VDC output 0, J6 24VDC output 1, J7 24VDC output 2, J8 24VDC output 3, J9 24VDC output 4, Q1 Q_NMOS_GDS, Q10 BS170, Q11 BS170, Q12 BS170, Q2 Q_NMOS_GDS, Q3 Q_NMOS_GDS, Q4 Q_NMOS_GDS, Q5 Q_NMOS_GDS, Q6 Q_NMOS_GDS, Q7 BS170, Q8 BS170, Q9 BS170, SW1 Rotary_Encoder_Switch, U1 ESP32-DEVKITC-32D, U2 PCA9685PW

Commit message: PCB v1
Connections:
- net 5VDC_output0: no longer R15.2, R16.2, R17.2, R18.2, R19.2, R20.2, R21.2, R22.2, R23.2, R24.2
- net 5VDC_output1: now also R15.2, R16.2
- net 5VDC_output2: now also R17.2, R18.2
- net 5VDC_output3: now also R19.2, R20.2
- net LEDcon0: now also U2.21 (LED14); no longer U2.19 (LED12)
- net stepperErr: now also U2.20 (LED13); no longer U2.18 (LED11)
- net stepperON: now also U2.19 (LED12); no longer U2.17 (LED10)
- new net 5VDC_output4: R21.2, R22.2, U2.17 (LED10)
- new net 5VDC_output5: R23.2, R24.2, U2.18 (LED11)
Changed lines of the file:
@@
 Text GLabel 11700 4650 2    50   Input ~ 0
 tempMeasure0
-Text GLabel 9200 4400 2    50   Input ~ 0
+Text GLabel 9200 4600 2    50   Input ~ 0
 stepperON
-Text GLabel 9200 4500 2    50   Input ~ 0
+Text GLabel 9200 4700 2    50   Input ~ 0
 stepperErr
 Text GLabel 11150 1150 0    50   Input ~ 0
@@
 Text GLabel 15300 7150 3    50   Input ~ 0
 reflectivesensor0
-Text GLabel 9200 4600 2    50   Input ~ 0
+Text GLabel 9200 4800 2    50   Input ~ 0
 LEDcon0
 Text GLabel 15250 6750 2    50   Input ~ 0
@@
 	5750 2900 5800 2900
 Text GLabel 5350 2900 0    50   Input ~ 0
-5VDC_output0
+5VDC_output1
 Connection ~ 5450 2900
 Wire Wire Line
@@
 	5750 4400 5800 4400
 Text GLabel 5350 4400 0    50   Input ~ 0
-5VDC_output0
+5VDC_output2
 Connection ~ 5450 4400
 Wire Wire Line
@@
 	5750 5900 5800 5900
 Text GLabel 5350 5900 0    50   Input ~ 0
-5VDC_output0
+5VDC_output3
 Connection ~ 5450 5900
 Wire Wire Line
@@
 	5750 7400 5800 7400
 Text GLabel 5350 7400 0    50   Input ~ 0
-5VDC_output0
+5VDC_output4
 Connection ~ 5450 7400
 Wire Wire Line
@@
 	5750 8900 5800 8900
 Text GLabel 5350 8900 0    50   Input ~ 0
-5VDC_output0
+5VDC_output5
 Connection ~ 5450 8900
 Wire Wire Line
@@
 	9150 4600 9200 4600
 Wire Wire Line
-	9150 4500 9200 4500
-Wire Wire Line
-	9150 4400 9200 4400
-Wire Wire Line
 	9150 4300 9200 4300
 Wire Wire Line
@@
 	0    -1   -1   0
 $EndComp
+Wire Wire Line
+	9200 4700 9150 4700
+Wire Wire Line
+	9150 4800 9200 4800
+Text GLabel 9200 4400 2    50   Input ~ 0
+5VDC_output4
+Text GLabel 9200 4500 2    50   Input ~ 0
+5VDC_output5
+Wire Wire Line
+	9200 4400 9150 4400
+Wire Wire Line
+	9150 4500 9200 4500
 $EndSCHEMATC

Commit message: PCB changes
Parts:
- removed C10, C11: 100uF, Capacitor_THT:CP_Radial_D6.3mm_P2.50mm, symbol Device:C
- removed R34, R35: 10k, Resistor_SMD:R_1206_3216Metric_Pad1.30x1.75mm_HandSolder, symbol Device:R
- removed SW1: Rotary_Encoder_Switch, Rotary_Encoder:RotaryEncoder_Alps_EC11E-Switch_Vertical_H20mm, symbol Device:Rotary_Encoder_Switch
- added J42: Conn_01x05_Male, Connector_PinHeader_2.54mm:PinHeader_1x05_P2.54mm_Vertical, symbol Connector:Conn_01x05_Male
Connections:
- net +3V3: now also C8.2, J42.4 (Pin_4); no longer C8.1
- net AO: now also J25.2 (Pin_2)
- net DT: now also J24.3 (Pin_3)
- net GND: now also J42.2 (Pin_2)
- net button: now also C8.1, J42.5 (Pin_5); no longer C8.2
- net enca: now also C12.2, J42.1 (Pin_1); no longer C13.1
- net encb: now also C13.1, J42.3 (Pin_3); no longer C12.2
- no-connect marks 1 -> 0
Other:
- moved on the sheet: C12, C13, C8
Changed lines of the file:
@@
 Text GLabel 9200 3400 2    50   Input ~ 0
 24VDC_output0
-NoConn ~ 1650 50
 $Comp
 L Device:R R27
@@
 Wire Wire Line
 	15000 2550 15200 2550
-$Comp
-L Device:Rotary_Encoder_Switch SW1
-U 1 1 61EAADC5
-P 13400 4800
-F 0 "SW1" H 13400 5167 50  0000 C CNN
-F 1 "Rotary_Encoder_Switch" H 13400 5076 50  0000 C CNN
-F 2 "Rotary_Encoder:RotaryEncoder_Alps_EC11E-Switch_Vertical_H20mm" H 13250 4960 50  0001 C CNN
-F 3 "~" H 13400 5060 50  0001 C CNN
-	1    13400 4800
-	-1   0    0    1
-$EndComp
-$Comp
-L power:GND #PWR073
-U 1 1 61EABB57
-P 14000 4800
-F 0 "#PWR073" H 14000 4550 50  0001 C CNN
-F 1 "GND" V 14005 4672 50  0000 R CNN
-F 2 "" H 14000 4800 50  0001 C CNN
-F 3 "" H 14000 4800 50  0001 C CNN
-	1    14000 4800
-	0    -1   -1   0
-$EndComp
-Text GLabel 13800 5100 3    50   Input ~ 0
+Text GLabel 13450 4400 1    50   Input ~ 0
 enca
-Text GLabel 13800 4500 1    50   Input ~ 0
+Text GLabel 13450 4600 3    50   Input ~ 0
 encb
-Text GLabel 12950 4650 1    50   Input ~ 0
+Text GLabel 13000 5000 3    50   Input ~ 0
 button
 Text GLabel 9200 3900 2    50   Input ~ 0
@@
 Text GLabel 9300 1750 2    50   Input ~ 0
 STEP0
-Wire Wire Line
-	13400 7850 13100 7850
-Wire Wire Line
-	13850 7850 13750 7850
-$Comp
-L Device:C C10
-U 1 1 6283E2CF
-P 13750 8000
-F 0 "C10" H 13865 8046 50  0000 L CNN
-F 1 "100uF" H 13865 7955 50  0000 L CNN
-F 2 "Capacitor_THT:CP_Radial_D6.3mm_P2.50mm" H 13788 7850 50  0001 C CNN
-F 3 "~" H 13750 8000 50  0001 C CNN
-	1    13750 8000
-	1    0    0    -1
-$EndComp
-$Comp
-L power:GND #PWR068
-U 1 1 6283E2C9
-P 13750 8150
-F 0 "#PWR068" H 13750 7900 50  0001 C CNN
-F 1 "GND" H 13755 7977 50  0000 C CNN
-F 2 "" H 13750 8150 50  0001 C CNN
-F 3 "" H 13750 8150 50  0001 C CNN
-	1    13750 8150
-	1    0    0    -1
-$EndComp
-$Comp
-L Device:R R34
-U 1 1 6283E2C3
-P 13550 7850
-F 0 "R34" V 13343 7850 50  0000 C CNN
-F 1 "10k" V 13434 7850 50  0000 C CNN
-F 2 "Resistor_SMD:R_1206_3216Metric_Pad1.30x1.75mm_HandSolder" V 13480 7850 50  0001 C CNN
-F 3 "~" H 13550 7850 50  0001 C CNN
-	1    13550 7850
-	0    1    1    0
-$EndComp
-Text GLabel 13850 7850 2    50   Input ~ 0
+Text GLabel 13150 7850 2    50   Input ~ 0
 AO
 $Comp
@@
 $EndComp
 $Comp
-L power:+3.3V #PWR058
-U 1 1 61A76F30
-P 12950 4950
-F 0 "#PWR058" H 12950 4800 50  0001 C CNN
-F 1 "+3.3V" V 12965 5078 50  0000 L CNN
-F 2 "" H 12950 4950 50  0001 C CNN
-F 3 "" H 12950 4950 50  0001 C CNN
-	1    12950 4950
-	-1   0    0    1
-$EndComp
-$Comp
 L Device:C C8
 U 1 1 61B1A5D9
-P 12850 4800
-F 0 "C8" H 12735 4754 50  0000 R CNN
-F 1 "100n" H 12735 4845 50  0000 R CNN
-F 2 "Capacitor_SMD:C_0603_1608Metric_Pad1.08x0.95mm_HandSolder" H 12888 4650 50  0001 C CNN
-F 3 "~" H 12850 4800 50  0001 C CNN
-	1    12850 4800
+P 13100 4850
+F 0 "C8" H 12985 4804 50  0000 R CNN
+F 1 "100n" H 12985 4895 50  0000 R CNN
+F 2 "Capacitor_SMD:C_0603_1608Metric_Pad1.08x0.95mm_HandSolder" H 13138 4700 50  0001 C CNN
+F 3 "~" H 13100 4850 50  0001 C CNN
+	1    13100 4850
 	-1   0    0    1
 $EndComp
-Wire Wire Line
-	12850 4950 12950 4950
-Wire Wire Line
-	12950 4950 13100 4950
-Wire Wire Line
-	13100 4950 13100 4900
-Connection ~ 12950 4950
 $Comp
 L Device:C C13
 U 1 1 61BB01E8
-P 14000 4950
-F 0 "C13" H 13885 4904 50  0000 R CNN
-F 1 "100n" H 13885 4995 50  0000 R CNN
-F 2 "Capacitor_SMD:C_0603_1608Metric_Pad1.08x0.95mm_HandSolder" H 14038 4800 50  0001 C CNN
-F 3 "~" H 14000 4950 50  0001 C CNN
-	1    14000 4950
+P 13650 4650
+F 0 "C13" H 13535 4604 50  0000 R CNN
+F 1 "100n" H 13535 4695 50  0000 R CNN
+F 2 "Capacitor_SMD:C_0603_1608Metric_Pad1.08x0.95mm_HandSolder" H 13688 4500 50  0001 C CNN
+F 3 "~" H 13650 4650 50  0001 C CNN
+	1    13650 4650
 	-1   0    0    1
 $EndComp
@@
 L Device:C C12
 U 1 1 61BC5069
-P 14000 4650
-F 0 "C12" H 13885 4604 50  0000 R CNN
-F 1 "100n" H 13885 4695 50  0000 R CNN
-F 2 "Capacitor_SMD:C_0603_1608Metric_Pad1.08x0.95mm_HandSolder" H 14038 4500 50  0001 C CNN
-F 3 "~" H 14000 4650 50  0001 C CNN
-	1    14000 4650
+P 13650 4350
+F 0 "C12" H 13535 4304 50  0000 R CNN
+F 1 "100n" H 13535 4395 50  0000 R CNN
+F 2 "Capacitor_SMD:C_0603_1608Metric_Pad1.08x0.95mm_HandSolder" H 13688 4200 50  0001 C CNN
+F 3 "~" H 13650 4350 50  0001 C CNN
+	1    13650 4350
 	-1   0    0    1
 $EndComp
-Connection ~ 14000 4800
-Wire Wire Line
-	14000 5100 13700 5100
-Wire Wire Line
-	13700 5100 13700 4900
-Wire Wire Line
-	13700 4700 13700 4500
-Wire Wire Line
-	13700 4500 14000 4500
 $Comp
 L Diode:1N4007 D13
@@
 	0    1    1    0
 $EndComp
-Text GLabel 13900 6850 2    50   Input ~ 0
-DT
-Text GLabel 13300 6950 2    50   Input ~ 0
-SCK
 Wire Wire Line
 	13100 6750 13300 6750
 Wire Wire Line
-	13300 6950 13100 6950
-Wire Wire Line
 	13100 7050 13300 7050
 $Comp
-L power:GND #PWR069
-U 1 1 628CF8CD
-P 13850 7150
-F 0 "#PWR069" H 13850 6900 50  0001 C CNN
-F 1 "GND" H 13855 6977 50  0000 C CNN
-F 2 "" H 13850 7150 50  0001 C CNN
-F 3 "" H 13850 7150 50  0001 C CNN
-	1    13850 7150
-	1    0    0    -1
-$EndComp
-$Comp
-L Device:C C11
-U 1 1 628CF8D3
-P 13850 7000
-F 0 "C11" H 13965 7046 50  0000 L CNN
-F 1 "100uF" H 13965 6955 50  0000 L CNN
-F 2 "Capacitor_THT:CP_Radial_D6.3mm_P2.50mm" H 13888 6850 50  0001 C CNN
-F 3 "~" H 13850 7000 50  0001 C CNN
-	1    13850 7000
-	1    0    0    -1
-$EndComp
-Wire Wire Line
-	13900 6850 13850 6850
-Wire Wire Line
-	13500 6850 13100 6850
-$Comp
 L power:+24V #PWR072
 U 1 1 62A230CD
@@
 $EndComp
 Wire Wire Line
-	14000 4800 13700 4800
-Wire Wire Line
 	14900 6750 14650 6750
 Wire Wire Line
@@
 	11250 5400 11200 5400
 Wire Wire Line
-	12850 4650 13100 4650
-Wire Wire Line
-	13100 4650 13100 4700
-Wire Wire Line
 	7500 4400 7500 4300
 Connection ~ 7500 4400
 Connection ~ 7500 4300
 $Comp
-L Device:R R35
-U 1 1 62E169D6
-P 13650 6850
-F 0 "R35" V 13443 6850 50  0000 C CNN
-F 1 "10k" V 13534 6850 50  0000 C CNN
-F 2 "Resistor_SMD:R_1206_3216Metric_Pad1.30x1.75mm_HandSolder" V 13580 6850 50  0001 C CNN
-F 3 "~" H 13650 6850 50  0001 C CNN
-	1    13650 6850
-	0    1    1    0
-$EndComp
-$Comp
 L Device:R R33
 U 1 1 62E2E02C
@@
 Wire Wire Line
 	15300 5800 15250 5800
-Connection ~ 13850 6850
-Wire Wire Line
-	13850 6850 13800 6850
 Wire Wire Line
 	15300 6850 15250 6850
@@
 Wire Wire Line
 	15250 7150 15350 7150
-Connection ~ 13750 7850
-Wire Wire Line
-	13750 7850 13700 7850
 Wire Wire Line
 	13150 7550 13100 7550
@@
 Wire Wire Line
 	9150 4500 9200 4500
+Text GLabel 13300 6850 2    50   Input ~ 0
+DT
+Text GLabel 13300 6950 2    50   Input ~ 0
+SCK
+Wire Wire Line
+	13300 6850 13100 6850
+Wire Wire Line
+	13300 6950 13100 6950
+Wire Wire Line
+	13150 7850 13100 7850
+$Comp
+L Connector:Conn_01x05_Male J42
+U 1 1 61FA40BF
+P 12750 4600
+F 0 "J42" H 12858 4981 50  0000 C CNN
+F 1 "Conn_01x05_Male" H 12858 4890 50  0000 C CNN
+F 2 "Connector_PinHeader_2.54mm:PinHeader_1x05_P2.54mm_Vertical" H 12750 4600 50  0001 C CNN
+F 3 "~" H 12750 4600 50  0001 C CNN
+	1    12750 4600
+	1    0    0    -1
+$EndComp
+$Comp
+L power:GND #PWR068
+U 1 1 61FA6407
+P 13650 4500
+F 0 "#PWR068" H 13650 4250 50  0001 C CNN
+F 1 "GND" V 13655 4372 50  0000 R CNN
+F 2 "" H 13650 4500 50  0001 C CNN
+F 3 "" H 13650 4500 50  0001 C CNN
+	1    13650 4500
+	0    -1   -1   0
+$EndComp
+Connection ~ 13650 4500
+Wire Wire Line
+	13650 4500 12950 4500
+Wire Wire Line
+	13550 4800 13550 4600
+Wire Wire Line
+	13550 4600 12950 4600
+Wire Wire Line
+	13550 4200 13550 4400
+Wire Wire Line
+	13550 4400 12950 4400
+$Comp
+L power:+3.3V #PWR058
+U 1 1 6243C181
+P 13250 4700
+F 0 "#PWR058" H 13250 4550 50  0001 C CNN
+F 1 "+3.3V" V 13265 4828 50  0000 L CNN
+F 2 "" H 13250 4700 50  0001 C CNN
+F 3 "" H 13250 4700 50  0001 C CNN
+	1    13250 4700
+	0    1    1    0
+$EndComp
+Wire Wire Line
+	13250 4700 13100 4700
+Connection ~ 13100 4700
+Wire Wire Line
+	13100 4700 12950 4700
+Wire Wire Line
+	13100 5000 12950 5000
+Wire Wire Line
+	12950 5000 12950 4800
+Wire Wire Line
+	13550 4800 13650 4800
+Wire Wire Line
+	13550 4200 13650 4200
 $EndSCHEMATC

Commit message: added routs
Parts:
- added H1, H2, H3, H4: MountingHole, MountingHole:MountingHole_3.2mm_M3, symbol Mechanical:MountingHole
- D1, D10, D11, D12, D13, D14, D2, D3, D4, D5, D6, D7, D8, D9: footprint Diode_SMD:D_SMA_Handsoldering -> Diode_THT:D_DO-15_P2.54mm_Vertical_AnodeUp
- J10, J11, J12, J13, J14, J15, J16, J17, J18, J26, J5, J6, J7, J8, J9: footprint TerminalBlock_4Ucon:TerminalBlock_4Ucon_1x02_P3.50mm_Horizontal -> TerminalBlock:TerminalBlock_bornier-2_P5.08mm
Connections:
- net 24VDC_output0: now also U2.8 (LED2); no longer U2.6 (LED0)
- net 24VDC_output1: now also U2.9 (LED3); no longer U2.7 (LED1)
- net 24VDC_output2: now also U2.10 (LED4); no longer U2.8 (LED2)
- net 24VDC_output3: now also U2.11 (LED5); no longer U2.9 (LED3)
- net 24VDC_output4: now also U2.12 (LED6); no longer U2.10 (LED4)
- net 24VDC_output5: now also U2.13 (LED7); no longer U2.11 (LED5)
- net 5VDC_output0: now also U2.15 (LED8); no longer U2.12 (LED6)
- net 5VDC_output1: now also U2.16 (LED9); no longer U2.13 (LED7)
- net 5VDC_output2: now also U2.17 (LED10); no longer U2.15 (LED8)
- net 5VDC_output3: now also U2.18 (LED11); no longer U2.16 (LED9)
- net 5VDC_output4: now also U2.6 (LED0); no longer U2.17 (LED10)
- net 5VDC_output5: now also U2.7 (LED1); no longer U2.18 (LED11)

Commit message: routs added
Parts:
- J10: value 24VDC output 5 -> 24VDCout5
- J11: value 5VDC output 0 -> 5VDCout0
- J12: value 5VDC output 1 -> 5VDCout1
- J13: value 5VDC output 2 -> 5VDCout2
- J14: value 5VDC output 3 -> 5VDCout3
- J15: value 5VDC output 4 -> 5VDCout4
- J16: value 5VDC output 5 -> 5VDCout5
- J5: value 24VDC output 0 -> 24VDCout0
- J6: value 24VDC output 1 -> 24VDCout1
- J7: value 24VDC output 2 -> 24VDCout2
- J8: value 24VDC output 3 -> 24VDCout3
- J9: value 24VDC output 4 -> 24VDCout4
Other:
- moved on the sheet: C16
Changed lines of the file:
@@
 P 4350 8500
 F 0 "J10" H 4430 8492 50  0000 L CNN
-F 1 "24VDC output 5" H 4430 8401 50  0000 L CNN
+F 1 "24VDCout5" H 4430 8401 50  0000 L CNN
 F 2 "TerminalBlock:TerminalBlock_bornier-2_P5.08mm" H 4350 8500 50  0001 C CNN
 F 3 "~" H 4350 8500 50  0001 C CNN
@@
 P 4350 7000
 F 0 "J9" H 4430 6992 50  0000 L CNN
-F 1 "24VDC output 4" H 4430 6901 50  0000 L CNN
+F 1 "24VDCout4" H 4430 6901 50  0000 L CNN
 F 2 "TerminalBlock:TerminalBlock_bornier-2_P5.08mm" H 4350 7000 50  0001 C CNN
 F 3 "~" H 4350 7000 50  0001 C CNN
@@
 P 4350 5500
 F 0 "J8" H 4430 5492 50  0000 L CNN
-F 1 "24VDC output 3" H 4430 5401 50  0000 L CNN
+F 1 "24VDCout3" H 4430 5401 50  0000 L CNN
 F 2 "TerminalBlock:TerminalBlock_bornier-2_P5.08mm" H 4350 5500 50  0001 C CNN
 F 3 "~" H 4350 5500 50  0001 C CNN
@@
 P 4350 4000
 F 0 "J7" H 4430 3992 50  0000 L CNN
-F 1 "24VDC output 2" H 4430 3901 50  0000 L CNN
+F 1 "24VDCout2" H 4430 3901 50  0000 L CNN
 F 2 "TerminalBlock:TerminalBlock_bornier-2_P5.08mm" H 4350 4000 50  0001 C CNN
 F 3 "~" H 4350 4000 50  0001 C CNN
@@
 P 4350 2500
 F 0 "J6" H 4430 2492 50  0000 L CNN
-F 1 "24VDC output 1" H 4430 2401 50  0000 L CNN
+F 1 "24VDCout1" H 4430 2401 50  0000 L CNN
 F 2 "TerminalBlock:TerminalBlock_bornier-2_P5.08mm" H 4350 2500 50  0001 C CNN
 F 3 "~" H 4350 2500 50  0001 C CNN
@@
 P 4350 1000
 F 0 "J5" H 4430 992 50  0000 L CNN
-F 1 "24VDC output 0" H 4430 901 50  0000 L CNN
+F 1 "24VDCout0" H 4430 901 50  0000 L CNN
 F 2 "TerminalBlock:TerminalBlock_bornier-2_P5.08mm" H 4350 1000 50  0001 C CNN
 F 3 "~" H 4350 1000 50  0001 C CNN
@@
 L Device:C C16
 U 1 1 622E7837
-P 15500 7150
-F 0 "C16" V 15248 7150 50  0000 C CNN
-F 1 "100uF" V 15339 7150 50  0000 C CNN
-F 2 "Capacitor_THT:CP_Radial_D6.3mm_P2.50mm" H 15538 7000 50  0001 C CNN
-F 3 "~" H 15500 7150 50  0001 C CNN
-	1    15500 7150
-	0    1    1    0
+P 15250 7400
+F 0 "C16" V 14998 7400 50  0000 C CNN
+F 1 "100uF" V 15089 7400 50  0000 C CNN
+F 2 "Capacitor_THT:CP_Radial_D6.3mm_P2.50mm" H 15288 7250 50  0001 C CNN
+F 3 "~" H 15250 7400 50  0001 C CNN
+	1    15250 7400
+	-1   0    0    1
 $EndComp
 $Comp
 L power:GND #PWR0108
 U 1 1 62301A12
-P 15650 7150
-F 0 "#PWR0108" H 15650 6900 50  0001 C CNN
-F 1 "GND" V 15655 7022 50  0000 R CNN
-F 2 "" H 15650 7150 50  0001 C CNN
-F 3 "" H 15650 7150 50  0001 C CNN
-	1    15650 7150
-	0    -1   -1   0
-$EndComp
-Text GLabel 15300 7150 3    50   Input ~ 0
+P 15250 7550
+F 0 "#PWR0108" H 15250 7300 50  0001 C CNN
+F 1 "GND" V 15255 7422 50  0000 R CNN
+F 2 "" H 15250 7550 50  0001 C CNN
+F 3 "" H 15250 7550 50  0001 C CNN
+	1    15250 7550
+	1    0    0    -1
+$EndComp
+Text GLabel 15250 7200 2    50   Input ~ 0
 reflectivesensor0
 Text GLabel 9200 4800 2    50   Input ~ 0
@@
 P 6300 1000
 F 0 "J11" H 6380 992 50  0000 L CNN
-F 1 "5VDC output 0" H 6380 901 50  0000 L CNN
+F 1 "5VDCout0" H 6380 901 50  0000 L CNN
 F 2 "TerminalBlock:TerminalBlock_bornier-2_P5.08mm" H 6300 1000 50  0001 C CNN
 F 3 "~" H 6300 1000 50  0001 C CNN
@@
 P 6300 2500
 F 0 "J12" H 6380 2492 50  0000 L CNN
-F 1 "5VDC output 1" H 6380 2401 50  0000 L CNN
+F 1 "5VDCout1" H 6380 2401 50  0000 L CNN
 F 2 "TerminalBlock:TerminalBlock_bornier-2_P5.08mm" H 6300 2500 50  0001 C CNN
 F 3 "~" H 6300 2500 50  0001 C CNN
@@
 P 6300 4000
 F 0 "J13" H 6380 3992 50  0000 L CNN
-F 1 "5VDC output 2" H 6380 3901 50  0000 L CNN
+F 1 "5VDCout2" H 6380 3901 50  0000 L CNN
 F 2 "TerminalBlock:TerminalBlock_bornier-2_P5.08mm" H 6300 4000 50  0001 C CNN
 F 3 "~" H 6300 4000 50  0001 C CNN
@@
 P 6300 5500
 F 0 "J14" H 6380 5492 50  0000 L CNN
-F 1 "5VDC output 3" H 6380 5401 50  0000 L CNN
+F 1 "5VDCout3" H 6380 5401 50  0000 L CNN
 F 2 "TerminalBlock:TerminalBlock_bornier-2_P5.08mm" H 6300 5500 50  0001 C CNN
 F 3 "~" H 6300 5500 50  0001 C CNN
@@
 P 6300 7000
 F 0 "J15" H 6380 6992 50  0000 L CNN
-F 1 "5VDC output 4" H 6380 6901 50  0000 L CNN
+F 1 "5VDCout4" H 6380 6901 50  0000 L CNN
 F 2 "TerminalBlock:TerminalBlock_bornier-2_P5.08mm" H 6300 7000 50  0001 C CNN
 F 3 "~" H 6300 7000 50  0001 C CNN
@@
 P 6300 8500
 F 0 "J16" H 6380 8492 50  0000 L CNN
-F 1 "5VDC output 5" H 6380 8401 50  0000 L CNN
+F 1 "5VDCout5" H 6380 8401 50  0000 L CNN
 F 2 "TerminalBlock:TerminalBlock_bornier-2_P5.08mm" H 6300 8500 50  0001 C CNN
 F 3 "~" H 6300 8500 50  0001 C CNN
@@
 Connection ~ 15250 6850
 Wire Wire Line
-	15250 7150 15350 7150
+	15250 7150 15250 7250
 Wire Wire Line
 	13150 7550 13100 7550
