File: main_board/main_board.sch (KiCad schematic (older format))
At the start: 134 parts, among them J1 stepper0, J10 24VDCout5, J11 5VDCout0, J12 5VDCout1, J13 5VDCout2, J14 5VDCout3, J15 5VDCout4, J16 5VDCout5, J17 temp0, J18 temp1, J19 I2C, J2 stepper1, J20 I2C, J21 I2C, J22 I2C, J23 analogIn0, J24 weightSensor, J25 lightSensor, J26 24VDC_in, J27 24VDC to 5VDC step down, J28 24VDC, J29 24VDC, J3 stepper2, J30 24VDC, J31 5VDC, J32 5VDC, J33 5VDC, J34 analogIn1, J35 reflectiveSensor, J36 24VDC, J37 24VDC, J38 24VDC, J39 5VDC, J4 stepper3, J40 5VDC, J41 5VDC, J42 encoder, J5 24VDCout0, J6 24VDCout1, J7 24VDCout2, J8 24VDCout3, J9 24VDCout4, Q1 Q_NMOS_GDS, Q10 BS170, Q11 BS170, Q12 BS170, Q2 Q_NMOS_GDS, Q3 Q_NMOS_GDS, Q4 Q_NMOS_GDS, Q5 Q_NMOS_GDS, Q6 Q_NMOS_GDS, Q7 BS170, Q8 BS170, Q9 BS170, U1 ESP32-DEVKITC-32D, U2 PCA9685PW

Commit message: software
Parts:
- R29, R30: value 10K -> 10k
- R35: value R -> 150R
Changed lines of the file:
@@
 P 11400 1000
 F 0 "R29" V 11193 1000 50  0000 C CNN
-F 1 "10K" V 11284 1000 50  0000 C CNN
+F 1 "10k" V 11284 1000 50  0000 C CNN
 F 2 "Resistor_SMD:R_1206_3216Metric_Pad1.30x1.75mm_HandSolder" V 11330 1000 50  0001 C CNN
 F 3 "~" H 11400 1000 50  0001 C CNN
@@
 P 11400 1150
 F 0 "R30" V 11193 1150 50  0000 C CNN
-F 1 "10K" V 11284 1150 50  0000 C CNN
+F 1 "10k" V 11284 1150 50  0000 C CNN
 F 2 "Resistor_SMD:R_1206_3216Metric_Pad1.30x1.75mm_HandSolder" V 11330 1150 50  0001 C CNN
 F 3 "~" H 11400 1150 50  0001 C CNN
@@
 P 9750 4900
 F 0 "R35" V 9543 4900 50  0000 C CNN
-F 1 "R" V 9634 4900 50  0000 C CNN
+F 1 "150R" V 9634 4900 50  0000 C CNN
 F 2 "Resistor_SMD:R_1206_3216Metric_Pad1.30x1.75mm_HandSolder" V 9680 4900 50  0001 C CNN
 F 3 "~" H 9750 4900 50  0001 C CNN

Commit message: problem s topenim
Parts:
- A1, A2, A3, A4: footprint Module:Pololu_Breakout-16_15.2x20.3mm -> main_board:Pololu_Breakout-16_15.2x20.3mm
- J10, J11, J12, J13, J14, J15, J16, J17, J18, J26, J5, J6, J7, J8, J9: footprint TerminalBlock:TerminalBlock_bornier-2_P5.08mm -> main_board:TerminalBlock_bornier-2_P5.08mm
- U1: footprint ESP32-DEVKITC-32D:MODULE_ESP32-DEVKITC-32D -> main_board:MODULE_ESP32-DEVKITC-32D
Changed lines of the file:
@@
 F 0 "J26" V 13064 512 50  0000 R CNN
 F 1 "24VDC_in" V 12973 512 50  0000 R CNN
-F 2 "TerminalBlock:TerminalBlock_bornier-2_P5.08mm" H 13100 700 50  0001 C CNN
+F 2 "main_board:TerminalBlock_bornier-2_P5.08mm" H 13100 700 50  0001 C CNN
 F 3 "~" H 13100 700 50  0001 C CNN
 	1    13100 700
@@
 F 0 "A1" H 1750 2331 50  0000 C CNN
 F 1 "Pololu_Breakout_DRV8825" H 1750 2240 50  0000 C CNN
-F 2 "Module:Pololu_Breakout-16_15.2x20.3mm" H 1950 750 50  0001 L CNN
+F 2 "main_board:Pololu_Breakout-16_15.2x20.3mm" H 1950 750 50  0001 L CNN
 F 3 "https://www.pololu.com/product/2982" H 1850 1250 50  0001 C CNN
 	1    1750 1550
@@
 F 0 "A2" H 1800 3981 50  0000 C CNN
 F 1 "Pololu_Breakout_DRV8825" H 1800 3890 50  0000 C CNN
-F 2 "Module:Pololu_Breakout-16_15.2x20.3mm" H 2000 2400 50  0001 L CNN
+F 2 "main_board:Pololu_Breakout-16_15.2x20.3mm" H 2000 2400 50  0001 L CNN
 F 3 "https://www.pololu.com/product/2982" H 1900 2900 50  0001 C CNN
 	1    1800 3200
@@
 F 0 "A3" H 1800 5631 50  0000 C CNN
 F 1 "Pololu_Breakout_DRV8825" H 1800 5540 50  0000 C CNN
-F 2 "Module:Pololu_Breakout-16_15.2x20.3mm" H 2000 4050 50  0001 L CNN
+F 2 "main_board:Pololu_Breakout-16_15.2x20.3mm" H 2000 4050 50  0001 L CNN
 F 3 "https://www.pololu.com/product/2982" H 1900 4550 50  0001 C CNN
 	1    1800 4850
@@
 F 0 "A4" H 1850 7281 50  0000 C CNN
 F 1 "Pololu_Breakout_DRV8825" H 1850 7190 50  0000 C CNN
-F 2 "Module:Pololu_Breakout-16_15.2x20.3mm" H 2050 5700 50  0001 L CNN
+F 2 "main_board:Pololu_Breakout-16_15.2x20.3mm" H 2050 5700 50  0001 L CNN
 F 3 "https://www.pololu.com/product/2982" H 1950 6200 50  0001 C CNN
 	1    1850 6500
@@
 F 0 "U1" H 8450 2917 50  0000 C CNN
 F 1 "ESP32-DEVKITC-32D" H 8450 2826 50  0000 C CNN
-F 2 "ESP32-DEVKITC-32D:MODULE_ESP32-DEVKITC-32D" H 8450 1750 50  0001 L BNN
+F 2 "main_board:MODULE_ESP32-DEVKITC-32D" H 8450 1750 50  0001 L BNN
 F 3 "" H 8450 1750 50  0001 L BNN
 F 4 "Espressif Systems" H 8450 1750 50  0001 L BNN "MANUFACTURER"
@@
 F 0 "J10" H 4430 8492 50  0000 L CNN
 F 1 "24VDCout5" H 4430 8401 50  0000 L CNN
-F 2 "TerminalBlock:TerminalBlock_bornier-2_P5.08mm" H 4350 8500 50  0001 C CNN
+F 2 "main_board:TerminalBlock_bornier-2_P5.08mm" H 4350 8500 50  0001 C CNN
 F 3 "~" H 4350 8500 50  0001 C CNN
 	1    4350 8500
@@
 F 0 "J9" H 4430 6992 50  0000 L CNN
 F 1 "24VDCout4" H 4430 6901 50  0000 L CNN
-F 2 "TerminalBlock:TerminalBlock_bornier-2_P5.08mm" H 4350 7000 50  0001 C CNN
+F 2 "main_board:TerminalBlock_bornier-2_P5.08mm" H 4350 7000 50  0001 C CNN
 F 3 "~" H 4350 7000 50  0001 C CNN
 	1    4350 7000
@@
 F 0 "J8" H 4430 5492 50  0000 L CNN
 F 1 "24VDCout3" H 4430 5401 50  0000 L CNN
-F 2 "TerminalBlock:TerminalBlock_bornier-2_P5.08mm" H 4350 5500 50  0001 C CNN
+F 2 "main_board:TerminalBlock_bornier-2_P5.08mm" H 4350 5500 50  0001 C CNN
 F 3 "~" H 4350 5500 50  0001 C CNN
 	1    4350 5500
@@
 F 0 "J7" H 4430 3992 50  0000 L CNN
 F 1 "24VDCout2" H 4430 3901 50  0000 L CNN
-F 2 "TerminalBlock:TerminalBlock_bornier-2_P5.08mm" H 4350 4000 50  0001 C CNN
+F 2 "main_board:TerminalBlock_bornier-2_P5.08mm" H 4350 4000 50  0001 C CNN
 F 3 "~" H 4350 4000 50  0001 C CNN
 	1    4350 4000
@@
 F 0 "J6" H 4430 2492 50  0000 L CNN
 F 1 "24VDCout1" H 4430 2401 50  0000 L CNN
-F 2 "TerminalBlock:TerminalBlock_bornier-2_P5.08mm" H 4350 2500 50  0001 C CNN
+F 2 "main_board:TerminalBlock_bornier-2_P5.08mm" H 4350 2500 50  0001 C CNN
 F 3 "~" H 4350 2500 50  0001 C CNN
 	1    4350 2500
@@
 F 0 "J5" H 4430 992 50  0000 L CNN
 F 1 "24VDCout0" H 4430 901 50  0000 L CNN
-F 2 "TerminalBlock:TerminalBlock_bornier-2_P5.08mm" H 4350 1000 50  0001 C CNN
+F 2 "main_board:TerminalBlock_bornier-2_P5.08mm" H 4350 1000 50  0001 C CNN
 F 3 "~" H 4350 1000 50  0001 C CNN
 	1    4350 1000
@@
 F 0 "J17" H 10730 4742 50  0000 L CNN
 F 1 "temp0" H 10730 4651 50  0000 L CNN
-F 2 "TerminalBlock:TerminalBlock_bornier-2_P5.08mm" H 10650 4750 50  0001 C CNN
+F 2 "main_board:TerminalBlock_bornier-2_P5.08mm" H 10650 4750 50  0001 C CNN
 F 3 "~" H 10650 4750 50  0001 C CNN
 	1    10650 4750
@@
 F 0 "J18" H 10730 5492 50  0000 L CNN
 F 1 "temp1" H 10730 5401 50  0000 L CNN
-F 2 "TerminalBlock:TerminalBlock_bornier-2_P5.08mm" H 10650 5500 50  0001 C CNN
+F 2 "main_board:TerminalBlock_bornier-2_P5.08mm" H 10650 5500 50  0001 C CNN
 F 3 "~" H 10650 5500 50  0001 C CNN
 	1    10650 5500
@@
 F 0 "J11" H 6380 992 50  0000 L CNN
 F 1 "5VDCout0" H 6380 901 50  0000 L CNN
-F 2 "TerminalBlock:TerminalBlock_bornier-2_P5.08mm" H 6300 1000 50  0001 C CNN
+F 2 "main_board:TerminalBlock_bornier-2_P5.08mm" H 6300 1000 50  0001 C CNN
 F 3 "~" H 6300 1000 50  0001 C CNN
 	1    6300 1000
@@
 F 0 "J12" H 6380 2492 50  0000 L CNN
 F 1 "5VDCout1" H 6380 2401 50  0000 L CNN
-F 2 "TerminalBlock:TerminalBlock_bornier-2_P5.08mm" H 6300 2500 50  0001 C CNN
+F 2 "main_board:TerminalBlock_bornier-2_P5.08mm" H 6300 2500 50  0001 C CNN
 F 3 "~" H 6300 2500 50  0001 C CNN
 	1    6300 2500
@@
 F 0 "J13" H 6380 3992 50  0000 L CNN
 F 1 "5VDCout2" H 6380 3901 50  0000 L CNN
-F 2 "TerminalBlock:TerminalBlock_bornier-2_P5.08mm" H 6300 4000 50  0001 C CNN
+F 2 "main_board:TerminalBlock_bornier-2_P5.08mm" H 6300 4000 50  0001 C CNN
 F 3 "~" H 6300 4000 50  0001 C CNN
 	1    6300 4000
@@
 F 0 "J14" H 6380 5492 50  0000 L CNN
 F 1 "5VDCout3" H 6380 5401 50  0000 L CNN
-F 2 "TerminalBlock:TerminalBlock_bornier-2_P5.08mm" H 6300 5500 50  0001 C CNN
+F 2 "main_board:TerminalBlock_bornier-2_P5.08mm" H 6300 5500 50  0001 C CNN
 F 3 "~" H 6300 5500 50  0001 C CNN
 	1    6300 5500
@@
 F 0 "J15" H 6380 6992 50  0000 L CNN
 F 1 "5VDCout4" H 6380 6901 50  0000 L CNN
-F 2 "TerminalBlock:TerminalBlock_bornier-2_P5.08mm" H 6300 7000 50  0001 C CNN
+F 2 "main_board:TerminalBlock_bornier-2_P5.08mm" H 6300 7000 50  0001 C CNN
 F 3 "~" H 6300 7000 50  0001 C CNN
 	1    6300 7000
@@
 F 0 "J16" H 6380 8492 50  0000 L CNN
 F 1 "5VDCout5" H 6380 8401 50  0000 L CNN
-F 2 "TerminalBlock:TerminalBlock_bornier-2_P5.08mm" H 6300 8500 50  0001 C CNN
+F 2 "main_board:TerminalBlock_bornier-2_P5.08mm" H 6300 8500 50  0001 C CNN
 F 3 "~" H 6300 8500 50  0001 C CNN
 	1    6300 8500
