File: main_board/main_board.kicad_pcb (KiCad board)
At the start: 2 copper layers, 145 x 87 mm, 135 parts, among them J1 stepper0, J10 24VDCout5, J11 5VDCout0, J12 5VDCout1, J13 5VDCout2, J14 5VDCout3, J15 5VDCout4, J16 5VDCout5, J17 temp0, J18 temp1, J19 I2C, J2 stepper1, J20 I2C, J21 I2C, J22 I2C, J23 analogIn0, J24 weightSensor, J25 lightSensor, J26 24VDC_in, J27 24VDC to 5VDC step down, J28 24VDC, J29 24VDC, J3 stepper2, J30 24VDC, J31 5VDC, J32 5VDC, J33 5VDC, J34 analogIn1, J35 reflectiveSensor, J36 24VDC, J37 24VDC, J38 24VDC, J39 5VDC, J4 stepper3, J40 5VDC, J41 5VDC, J42 encoder, J5 24VDCout0, J6 24VDCout1, J7 24VDCout2, J8 24VDCout3, J9 24VDCout4, Q1 Q_NMOS_GDS, Q10 BS170, Q11 BS170, Q12 BS170, Q2 Q_NMOS_GDS, Q3 Q_NMOS_GDS, Q4 Q_NMOS_GDS, Q5 Q_NMOS_GDS, Q6 Q_NMOS_GDS, Q7 BS170, Q8 BS170, Q9 BS170, U1 ESP32-DEVKITC-32D, U2 PCA9685PW

Commit message: problems fix
Parts:
- added D16: LED, LED_THT:LED_D3.0mm, F.Cu at (135.9, 53.3)
- added R35: R, Resistor_SMD:R_1206_3216Metric_Pad1.30x1.75mm_HandSolder, F.Cu at (132.1, 52.1)
- C5: footprint Capacitor_THT:CP_Radial_D4.0mm_P1.50mm -> Capacitor_THT:CP_Radial_D6.3mm_P2.50mm
- J23, J34: footprint Connector_PinHeader_2.54mm:PinHeader_1x03_P2.54mm_Vertical -> Connector_PinHeader_2.54mm:PinHeader_1x04_P2.54mm_Vertical
- moved C9 17.1 mm to (113.0, 40.6)
- moved C15 17.1 mm to (100.3, 52.0)
- moved C5 4.58 mm to (106.7, 68.6)
- moved J23 2.54 mm to (106.7, 53.3)
- moved R29 2.00 mm to (103.9, 58.4)
- moved C7 1.80 mm to (81.3, 80.0), turned to 0 degrees
- moved C16 1.77 mm to (108.0, 19.1), turned to 0 degrees
- moved C6 1.77 mm to (71.1, 80.0), turned to 0 degrees
- moved J34 1.27 mm to (119.4, 40.6)
- moved J42 1.27 mm to (142.2, 55.9)
- moved C10 1.27 mm to (127.0, 25.4)
- moved J35 1.27 mm to (118.1, 19.1)
- moved R36 1.27 mm to (112.8, 26.7)
- moved C12 1.27 mm to (138.4, 59.3)
- moved C13 1.27 mm to (134.6, 59.3)
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Connections:
- net tempMeasure0 renamed temp0
- net tempMeasure1 renamed temp1
- C15 pad 1: hallmeasure1 -> Net-(C15-Pad1)
- C16 pad 1: GND -> reflectiveSensor0
- C16 pad 2: reflectivesensor0 -> GND
- C9 pad 1: hallmeasure0 -> Net-(C9-Pad1)
- J23 pad 1: +5V -> +3V3
- J23 pad 2: GND -> +5V
- J23 pad 3: Net-(J23-Pad3) -> GND
- J24 pad 1: +5V -> +3V3
- J25 pad 1: +5V -> +3V3
- J34 pad 1: +5V -> +3V3
- J34 pad 2: GND -> +5V
- J34 pad 3: Net-(J34-Pad3) -> GND
- R33 pad 1: Net-(J23-Pad3) -> Net-(J23-Pad4)
- R33 pad 2: hallmeasure0 -> analogIn0
- R37 pad 1: Net-(J34-Pad3) -> Net-(J34-Pad4)
- R37 pad 2: hallmeasure1 -> analogIn1
- R38 pad 2: reflectivesensor0 -> reflectiveSensor0
- U1 pad 10: DIR3 -> SCK
- U1 pad 12: Net-(R25-Pad1) -> DIR2
- U1 pad 15: hallmeasure1 -> encb
- U1 pad 20: Net-(U1-Pad20) -> GND
- U1 pad 26: Net-(U1-Pad26) -> GND
- U1 pad 27: DIR2 -> DT
- U1 pad 29: STEP0 -> DIR0
- U1 pad 3: hallmeasure0 -> analogIn0
- U1 pad 32: reflectivesensor0 -> button
- U1 pad 33: DIR0 -> STEP0
- U1 pad 35: Net-(R26-Pad1) -> DIR3
- U1 pad 4: encb -> analogIn1
- U1 pad 5: button -> reflectivesensor0
- U1 pad 7: DT -> Net-(R25-Pad1)
- U1 pad 8: SCK -> Net-(R26-Pad1)
Routing:
- net GND: track 0.00 -> 718.4 mm, vias 0 -> 30
- net +24V: track 0.00 -> 366.0 mm, vias 0 -> 1
- net +5V: track 0.00 -> 310.2 mm
- net stepperErr: track 0.00 -> 155.2 mm
- net +3V3: track 0.00 -> 149.9 mm, vias 0 -> 1
- net stepperON: track 0.00 -> 139.2 mm
- net button: track 0.00 -> 98.3 mm, vias 0 -> 1
- net SDA: track 0.00 -> 94.8 mm, vias 0 -> 1
- net enca: track 0.00 -> 91.4 mm, vias 0 -> 1
- net SCL: track 0.00 -> 84.6 mm, vias 0 -> 1
- net DT: track 0.00 -> 80.4 mm, vias 0 -> 1
- net encb: track 0.00 -> 76.8 mm, vias 0 -> 1
- net DIR3: track 0.00 -> 65.3 mm
- net STEP3: track 0.00 -> 61.4 mm, vias 0 -> 1
- net 24VDC_output5: track 0.00 -> 52.7 mm
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- added copper zone on B.Cu, net GND
- added copper zone on F.Cu, net GND

Commit message: bug fix
Routing:
- net reflectiveSensor0: track 0.00 -> 5.85 mm
- net reflectivesensor0: track 43.9 -> 38.1 mm
Changed lines of the file:
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@@
   (segment (start 107.99 19.05) (end 107.99 35.52) (width 0.25) (layer B.Cu) (net 52))
   (segment (start 107.99 35.52) (end 92.71 50.8) (width 0.25) (layer B.Cu) (net 52))
-  (segment (start 107.99 19.05) (end 107.99 20.1753) (width 0.25) (layer F.Cu) (net 52))
-  (segment (start 106.12 24.13) (end 106.12 22.0453) (width 0.25) (layer F.Cu) (net 52))
-  (segment (start 106.12 22.0453) (end 107.99 20.1753) (width 0.25) (layer F.Cu) (net 52))
   (segment (start 163.83 77.47) (end 163.83 78.9153) (width 0.25) (layer F.Cu) (net 53))
   (segment (start 163.9034 82.4766) (end 162.56 83.82) (width 0.25) (layer F.Cu) (net 53))
@@
   (segment (start 118.11 26.67) (end 114.3 26.67) (width 0.25) (layer F.Cu) (net 73))
   (segment (start 109.22 24.13) (end 109.22 29.21) (width 0.25) (layer F.Cu) (net 74))
-  (segment (start 118.11 24.13) (end 109.22 24.13) (width 0.25) (layer F.Cu) (net 74))
+  (segment (start 109.22 24.13) (end 118.11 24.13) (width 0.25) (layer F.Cu) (net 74))
   (segment (start 160.02 83.82) (end 160.02 78.74) (width 0.25) (layer F.Cu) (net 75))
   (segment (start 160.02 78.74) (end 158.75 77.47) (width 0.25) (layer F.Cu) (net 75))
@@
   (segment (start 110.1996 35.8504) (end 110.1996 33.02) (width 0.25) (layer B.Cu) (net 117))
   (via (at 110.1996 33.02) (size 0.8) (layers F.Cu B.Cu) (net 117))
+  (segment (start 107.99 19.05) (end 107.99 20.28) (width 0.25) (layer F.Cu) (net 118))
+  (segment (start 106.12 22.15) (end 106.12 24.13) (width 0.25) (layer F.Cu) (net 118))
+  (segment (start 107.99 20.28) (end 106.12 22.15) (width 0.25) (layer F.Cu) (net 118))
   (segment (start 138.43 53.34) (end 137.2046 54.5654) (width 0.25) (layer F.Cu) (net 119))
   (segment (start 137.2046 54.5654) (end 133.0254 54.5654) (width 0.25) (layer F.Cu) (net 119))

Commit message: reroute
Parts:
- removed R25, R26: 330R, Resistor_SMD:R_1206_3216Metric_Pad1.30x1.75mm_HandSolder
- D15: value LED -> powerOn
- moved D15 1.27 mm to (135.9, 45.7)
- moved G*** 0.45 mm to (162.6, 88.9)
Connections:
- R34 pad 1: DIR1 -> STEP0
- U1 pad 13: DIR1 -> STEP0
- U1 pad 33: STEP0 -> DIR1
- U1 pad 5: reflectivesensor0 -> reflectiveSensor0
- U1 pad 7: Net-(R25-Pad1) -> temp0
- U1 pad 8: Net-(R26-Pad1) -> temp1
Routing:
- net temp0: track 10.7 -> 57.1 mm
- net 24VDC_output0: track 43.5 -> 85.7 mm
- net Net-(R25-Pad1): track 40.7 -> 0.00 mm, vias 1 -> 0
- net reflectivesensor0: track 38.1 -> 0.00 mm
- net temp1: track 10.7 -> 48.3 mm
- net Net-(R26-Pad1): track 37.5 -> 0.00 mm, vias 1 -> 0
- net reflectiveSensor0: track 5.85 -> 38.9 mm
- net button: track 98.3 -> 125.1 mm, vias 1 -> 0
- net STEP0: track 14.0 -> 40.2 mm
- net enca: track 91.4 -> 117.1 mm, vias 1 -> 0
- net DIR1: track 38.0 -> 13.2 mm
- net +24V: track 366.0 -> 389.0 mm, vias 1 -> 0
- net GND: track 718.4 -> 732.3 mm, vias 30 -> 43
- net LEDcon0: track 52.6 -> 39.0 mm, vias 0 -> 2
- net stepperErr: track 155.2 -> 142.1 mm
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Other:
- board text added: "Filament Recycler V1.0 12/21 Jan Cícha"
- board text removed: "Filament Recycler V1.0 Jan Cícha"

Commit message: reroute
Routing:
- net GND: track 732.3 -> 765.2 mm, vias 43 -> 23
- net 24VDC_output5: track 52.0 -> 82.7 mm
- net encb: track 77.8 -> 103.8 mm
- net +3V3: track 149.7 -> 167.0 mm, vias 1 -> 2
- net button: track 125.1 -> 109.7 mm, vias 0 -> 1
- net 5VDC_output1: track 28.8 -> 42.7 mm, vias 0 -> 2
- net 5VDC_output2: track 27.2 -> 37.1 mm
- net 5VDC_output3: track 28.7 -> 20.3 mm
- net +5V: track 319.1 -> 324.8 mm
- net 5VDC_output0: track 42.2 -> 37.3 mm, vias 0 -> 2
- net SDA: track 93.1 -> 88.8 mm, vias 1 -> 2
- net +24V: track 389.0 -> 393.2 mm
- net temp0: track 57.1 -> 60.8 mm
- net SCL: track 76.5 -> 80.1 mm
- net 24VDC_output2: track 41.0 -> 38.2 mm
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