File: main_board/main_board.kicad_pcb (KiCad board)
At the start: 2 copper layers, 145 x 87 mm, 135 parts, among them J1 stepper0, J10 24VDCout5, J11 5VDCout0, J12 5VDCout1, J13 5VDCout2, J14 5VDCout3, J15 5VDCout4, J16 5VDCout5, J17 temp0, J18 temp1, J19 I2C, J2 stepper1, J20 I2C, J21 I2C, J22 I2C, J23 analogIn0, J24 weightSensor, J25 lightSensor, J26 24VDC_in, J27 24VDC to 5VDC step down, J28 24VDC, J29 24VDC, J3 stepper2, J30 24VDC, J31 5VDC, J32 5VDC, J33 5VDC, J34 analogIn1, J35 reflectiveSensor, J36 24VDC, J37 24VDC, J38 24VDC, J39 5VDC, J4 stepper3, J40 5VDC, J41 5VDC, J42 encoder, J5 24VDCout0, J6 24VDCout1, J7 24VDCout2, J8 24VDCout3, J9 24VDCout4, Q1 Q_NMOS_GDS, Q10 BS170, Q11 BS170, Q12 BS170, Q2 Q_NMOS_GDS, Q3 Q_NMOS_GDS, Q4 Q_NMOS_GDS, Q5 Q_NMOS_GDS, Q6 Q_NMOS_GDS, Q7 BS170, Q8 BS170, Q9 BS170, U1 ESP32-DEVKITC-32D, U2 PCA9685PW

Commit message: software
Routing:
- net GND: vias 23 -> 28
- net (no net): vias 1 -> 0

Commit message: problem s topenim
Parts:
- A1, A2, A3, A4: footprint Module:Pololu_Breakout-16_15.2x20.3mm -> main_board:Pololu_Breakout-16_15.2x20.3mm
- J10, J11, J12, J13, J14, J15, J16, J17, J18, J26, J5, J6, J7, J8, J9: footprint TerminalBlock:TerminalBlock_bornier-2_P5.08mm -> main_board:TerminalBlock_bornier-2_P5.08mm
- R29, R30: value 10K -> 10k
- R35: value R -> 150R
- U1: footprint ESP32-DEVKITC-32D:MODULE_ESP32-DEVKITC-32D -> main_board:MODULE_ESP32-DEVKITC-32D
